Commit message: finish urdf files

File: src/robot_description/urdf/delta_robot.urdf (robot description, URDF)
Before this commit: robot delta_robot, 8 links, 7 joints
Links:
- link base_link: geometry collision mesh filename=package://robot_description/meshes/base_link.STL; visual mesh filename=package://robot_description/meshes/base_link.STL
- link end_effector: geometry collision mesh filename=package://robot_description/meshes/end_effector.STL; visual mesh filename=package://robot_description/meshes/end_effector.STL
- link lower_arm_link_1: geometry collision mesh filename=package://robot_description/meshes/lower_arm_link_1.STL; visual mesh filename=package://robot_description/meshes/lower_arm_link_1.STL
- link lower_arm_link_2: geometry collision mesh filename=package://robot_description/meshes/lower_arm_link_2.STL; visual mesh filename=package://robot_description/meshes/lower_arm_link_2.STL
- link lower_arm_link_3: geometry collision mesh filename=package://robot_description/meshes/lower_arm_link_3.STL; visual mesh filename=package://robot_description/meshes/lower_arm_link_3.STL
- link upper_arm_link_1: geometry collision mesh filename=package://robot_description/meshes/upper_arm_link_1.STL; visual mesh filename=package://robot_description/meshes/upper_arm_link_1.STL
- link upper_arm_link_2: geometry collision mesh filename=package://robot_description/meshes/upper_arm_link_2.STL; visual mesh filename=package://robot_description/meshes/upper_arm_link_2.STL
- link upper_arm_link_3: geometry collision mesh filename=package://robot_description/meshes/upper_arm_link_3.STL; visual mesh filename=package://robot_description/meshes/upper_arm_link_3.STL
Joints:
- joint lower_arm_joint_1: limit lower=0 upper=0 effort=0 velocity=0 -> lower=-1.57 upper=1.57 effort=5.0 velocity=1.0
- joint lower_arm_joint_2: limit lower=0 upper=0 effort=0 velocity=0 -> lower=-1.57 upper=1.57 effort=5.0 velocity=1.0
- joint lower_arm_joint_3: limit lower=0 upper=0 effort=0 velocity=0 -> lower=-1.57 upper=1.57 effort=5.0 velocity=1.0
- joint upper_arm_joint_1: limit lower=0 upper=0 effort=0 velocity=0 -> lower=-1.57 upper=1.57 effort=5.0 velocity=1.0
- joint upper_arm_joint_2: limit lower=0 upper=0 effort=0 velocity=0 -> lower=-1.57 upper=1.57 effort=5.0 velocity=1.0
- joint upper_arm_joint_3: limit lower=0 upper=0 effort=0 velocity=0 -> lower=-1.57 upper=1.57 effort=5.0 velocity=1.0
